File: CR-serial.kicad_sch (KiCad schematic)
At the start: 8 parts, among them J1 USB_B, U1 CP2108-xxx-xM, U3 ECMF02-4CMX8

Commit message: Fix ferrite bead footprint
Parts:
- FB1: footprint Inductor_SMD:L_0201_0603Metric -> Inductor_SMD:L_0603_1608Metric
Changed lines of the file:
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@@
 			)
 		)
-		(property "Footprint" "Inductor_SMD:L_0201_0603Metric"
+		(property "Footprint" "Inductor_SMD:L_0603_1608Metric"
 			(at 69.85 163.068 90)
 			(effects
